File: Boost_Board.sch (KiCad schematic (older format))
At the start: 7 parts

Commit message: done with layout
Parts:
- added C3, C4: C, Capacitor_SMD:C_0805_2012Metric_Pad1.15x1.40mm_HandSolder, symbol Device:C
- added J3, J4: Conn_01x02_Male, Connector_PinHeader_2.54mm:PinHeader_1x02_P2.54mm_Vertical, symbol Connector:Conn_01x02_Male
- added L3: L, Inductor_SMD:L_0805_2012Metric_Pad1.15x1.40mm_HandSolder, symbol Device:L
- added L4: L, Boost_Board:1008_Inductor, symbol Device:L
- added U2: TPS613221ADBVT, Package_TO_SOT_SMD:SOT-23-5_HandSoldering, symbol TPS613221ADBVT:TPS613221ADBVT
- C1, C2: renamed from C?; footprint (none) -> Capacitor_SMD:C_0805_2012Metric_Pad1.15x1.40mm_HandSolder
- L1: renamed from L?; footprint (none) -> Inductor_SMD:L_0805_2012Metric_Pad1.15x1.40mm_HandSolder
- L2: renamed from L?; footprint (none) -> Boost_Board:1008_Inductor
- U1: renamed from U?; footprint DBV5 -> Package_TO_SOT_SMD:SOT-23-5_HandSoldering
- gave numbers to parts that had none: 2
Connections:
- net GND: now also C3.2, C4.2, J3.2 (Pin_2), J4.2 (Pin_2), U2.2 (GND)
- new net: J3.1 (Pin_1), L3.1, L4.1
- new net: L3.2, L4.2, U2.1 (SW)
- new net: C3.1, C4.1, J4.1 (Pin_1), U2.4 (VOUT)
Changed lines of the file:
@@
 EESchema Schematic File Version 4
+LIBS:Boost_Board-cache
 EELAYER 29 0
 EELAYER END
@@
 $EndDescr
 $Comp
-L Device:L L?
+L Device:L L1
 U 1 1 5D072E2C
 P 2200 3150
-F 0 "L?" V 2390 3150 50  0000 C CNN
+F 0 "L1" V 2390 3150 50  0000 C CNN
 F 1 "L" V 2299 3150 50  0000 C CNN
-F 2 "" H 2200 3150 50  0001 C CNN
+F 2 "Inductor_SMD:L_0805_2012Metric_Pad1.15x1.40mm_HandSolder" H 2200 3150 50  0001 C CNN
 F 3 "~" H 2200 3150 50  0001 C CNN
 	1    2200 3150
@@
 $EndComp
 $Comp
-L Device:C C?
+L Device:C C1
 U 1 1 5D07330C
 P 4500 3600
-F 0 "C?" H 4615 3646 50  0000 L CNN
+F 0 "C1" H 4615 3646 50  0000 L CNN
 F 1 "C" H 4615 3555 50  0000 L CNN
-F 2 "" H 4538 3450 50  0001 C CNN
+F 2 "Capacitor_SMD:C_0805_2012Metric_Pad1.15x1.40mm_HandSolder" H 4538 3450 50  0001 C CNN
 F 3 "~" H 4500 3600 50  0001 C CNN
 	1    4500 3600
@@
 $EndComp
 $Comp
-L TPS613221ADBVT:TPS613221ADBVT U?
+L TPS613221ADBVT:TPS613221ADBVT U1
 U 1 1 5D0739C4
 P 2650 3350
-F 0 "U?" H 3450 3737 60  0000 C CNN
+F 0 "U1" H 3450 3737 60  0000 C CNN
 F 1 "TPS613221ADBVT" H 3450 3631 60  0000 C CNN
-F 2 "DBV5" H 3450 3590 60  0001 C CNN
-F 3 "" H 2650 3350 60  0000 C CNN
+F 2 "Package_TO_SOT_SMD:SOT-23-5_HandSoldering" H 3450 3590 60  0001 C CNN
+F 3 "https://www.ti.com/lit/ds/symlink/tps61322.pdf" H 2650 3350 60  0001 C CNN
 	1    2650 3350
 	1    0    0    -1
 $EndComp
 $Comp
-L Connector:Conn_01x02_Male J?
+L Connector:Conn_01x02_Male J1
 U 1 1 5D0747F6
 P 1100 3300
-F 0 "J?" H 1208 3481 50  0000 C CNN
+F 0 "J1" H 1208 3481 50  0000 C CNN
 F 1 "Conn_01x02_Male" H 1208 3390 50  0000 C CNN
 F 2 "Connector_PinHeader_2.54mm:PinHeader_1x02_P2.54mm_Vertical" H 1100 3300 50  0001 C CNN
@@
 $EndComp
 $Comp
-L Connector:Conn_01x02_Male J?
+L Connector:Conn_01x02_Male J2
 U 1 1 5D075422
 P 5600 3450
-F 0 "J?" H 5572 3424 50  0000 R CNN
+F 0 "J2" H 5572 3424 50  0000 R CNN
 F 1 "Conn_01x02_Male" H 5572 3333 50  0000 R CNN
 F 2 "Connector_PinHeader_2.54mm:PinHeader_1x02_P2.54mm_Vertical" H 5600 3450 50  0001 C CNN
@@
 $EndComp
 $Comp
-L Device:C C?
+L Device:C C2
 U 1 1 5D07603F
 P 4850 3600
-F 0 "C?" H 4965 3646 50  0000 L CNN
+F 0 "C2" H 4965 3646 50  0000 L CNN
 F 1 "C" H 4965 3555 50  0000 L CNN
-F 2 "" H 4888 3450 50  0001 C CNN
+F 2 "Capacitor_SMD:C_0805_2012Metric_Pad1.15x1.40mm_HandSolder" H 4888 3450 50  0001 C CNN
 F 3 "~" H 4850 3600 50  0001 C CNN
 	1    4850 3600
@@
 $EndComp
 $Comp
-L Device:L L?
+L Device:L L2
 U 1 1 5D07B6A4
 P 2200 3450
-F 0 "L?" V 2390 3450 50  0000 C CNN
+F 0 "L2" V 2390 3450 50  0000 C CNN
 F 1 "L" V 2299 3450 50  0000 C CNN
-F 2 "" H 2200 3450 50  0001 C CNN
+F 2 "Boost_Board:1008_Inductor" H 2200 3450 50  0001 C CNN
 F 3 "~" H 2200 3450 50  0001 C CNN
 	1    2200 3450
@@
 	1350 3400 1350 3650
 $Comp
-L power:GND #PWR?
+L power:GND #PWR0101
 U 1 1 5D07FCE3
 P 1350 3650
-F 0 "#PWR?" H 1350 3400 50  0001 C CNN
+F 0 "#PWR0101" H 1350 3400 50  0001 C CNN
 F 1 "GND" H 1355 3477 50  0000 C CNN
 F 2 "" H 1350 3650 50  0001 C CNN
@@
 	2550 3450 2550 3700
 $Comp
-L power:GND #PWR?
+L power:GND #PWR0102
 U 1 1 5D080818
 P 2550 3700
-F 0 "#PWR?" H 2550 3450 50  0001 C CNN
+F 0 "#PWR0102" H 2550 3450 50  0001 C CNN
 F 1 "GND" H 2555 3527 50  0000 C CNN
 F 2 "" H 2550 3700 50  0001 C CNN
@@
 	5150 3550 5150 3750
 $Comp
-L power:GND #PWR?
+L power:GND #PWR0103
 U 1 1 5D085DF8
 P 5150 3750
-F 0 "#PWR?" H 5150 3500 50  0001 C CNN
+F 0 "#PWR0103" H 5150 3500 50  0001 C CNN
 F 1 "GND" H 5155 3577 50  0000 C CNN
 F 2 "" H 5150 3750 50  0001 C CNN
@@
 	4700 3750 4850 3750
 $Comp
-L power:GND #PWR?
+L power:GND #PWR0104
 U 1 1 5D08918F
 P 4700 3900
-F 0 "#PWR?" H 4700 3650 50  0001 C CNN
+F 0 "#PWR0104" H 4700 3650 50  0001 C CNN
 F 1 "GND" H 4705 3727 50  0000 C CNN
 F 2 "" H 4700 3900 50  0001 C CNN
@@
 Wire Wire Line
 	4850 3450 5400 3450
+$Comp
+L Device:L L3
+U 1 1 5D0819B7
+P 2100 1800
+F 0 "L3" V 2290 1800 50  0000 C CNN
+F 1 "L" V 2199 1800 50  0000 C CNN
+F 2 "Inductor_SMD:L_0805_2012Metric_Pad1.15x1.40mm_HandSolder" H 2100 1800 50  0001 C CNN
+F 3 "~" H 2100 1800 50  0001 C CNN
+	1    2100 1800
+	0    -1   -1   0
+$EndComp
+$Comp
+L Device:C C3
+U 1 1 5D0819BD
+P 4400 2250
+F 0 "C3" H 4515 2296 50  0000 L CNN
+F 1 "C" H 4515 2205 50  0000 L CNN
+F 2 "Capacitor_SMD:C_0805_2012Metric_Pad1.15x1.40mm_HandSolder" H 4438 2100 50  0001 C CNN
+F 3 "~" H 4400 2250 50  0001 C CNN
+	1    4400 2250
+	1    0    0    -1
+$EndComp
+$Comp
+L TPS613221ADBVT:TPS613221ADBVT U2
+U 1 1 5D0819C3
+P 2550 2000
+F 0 "U2" H 3350 2387 60  0000 C CNN
+F 1 "TPS613221ADBVT" H 3350 2281 60  0000 C CNN
+F 2 "Package_TO_SOT_SMD:SOT-23-5_HandSoldering" H 3350 2240 60  0001 C CNN
+F 3 "https://www.ti.com/lit/ds/symlink/tps61322.pdf" H 2550 2000 60  0001 C CNN
+	1    2550 2000
+	1    0    0    -1
+$EndComp
+$Comp
+L Connector:Conn_01x02_Male J3
+U 1 1 5D0819C9
+P 1000 1950
+F 0 "J3" H 1108 2131 50  0000 C CNN
+F 1 "Conn_01x02_Male" H 1108 2040 50  0000 C CNN
+F 2 "Connector_PinHeader_2.54mm:PinHeader_1x02_P2.54mm_Vertical" H 1000 1950 50  0001 C CNN
+F 3 "~" H 1000 1950 50  0001 C CNN
+	1    1000 1950
+	1    0    0    -1
+$EndComp
+$Comp
+L Connector:Conn_01x02_Male J4
+U 1 1 5D0819CF
+P 5500 2100
+F 0 "J4" H 5472 2074 50  0000 R CNN
+F 1 "Conn_01x02_Male" H 5472 1983 50  0000 R CNN
+F 2 "Connector_PinHeader_2.54mm:PinHeader_1x02_P2.54mm_Vertical" H 5500 2100 50  0001 C CNN
+F 3 "~" H 5500 2100 50  0001 C CNN
+	1    5500 2100
+	-1   0    0    -1
+$EndComp
+$Comp
+L Device:C C4
+U 1 1 5D0819D5
+P 4750 2250
+F 0 "C4" H 4865 2296 50  0000 L CNN
+F 1 "C" H 4865 2205 50  0000 L CNN
+F 2 "Capacitor_SMD:C_0805_2012Metric_Pad1.15x1.40mm_HandSolder" H 4788 2100 50  0001 C CNN
+F 3 "~" H 4750 2250 50  0001 C CNN
+	1    4750 2250
+	1    0    0    -1
+$EndComp
+$Comp
+L Device:L L4
+U 1 1 5D0819DB
+P 2100 2100
+F 0 "L4" V 2290 2100 50  0000 C CNN
+F 1 "L" V 2199 2100 50  0000 C CNN
+F 2 "Boost_Board:1008_Inductor" H 2100 2100 50  0001 C CNN
+F 3 "~" H 2100 2100 50  0001 C CNN
+	1    2100 2100
+	0    -1   -1   0
+$EndComp
+Wire Wire Line
+	2550 2000 2350 2000
+Wire Wire Line
+	2350 2000 2350 1800
+Wire Wire Line
+	2350 2000 2350 2100
+Wire Wire Line
+	2350 2100 2250 2100
+Connection ~ 2350 2000
+Wire Wire Line
+	2350 1800 2250 1800
+Wire Wire Line
+	1950 1800 1750 1800
+Wire Wire Line
+	1750 1800 1750 1950
+Wire Wire Line
+	1750 2100 1950 2100
+Wire Wire Line
+	1200 1950 1750 1950
+Connection ~ 1750 1950
+Wire Wire Line
+	1750 1950 1750 2100
+Wire Wire Line
+	1200 2050 1250 2050
+Wire Wire Line
+	1250 2050 1250 2300
+$Comp
+L power:GND #PWR01
+U 1 1 5D0819EF
+P 1250 2300
+F 0 "#PWR01" H 1250 2050 50  0001 C CNN
+F 1 "GND" H 1255 2127 50  0000 C CNN
+F 2 "" H 1250 2300 50  0001 C CNN
+F 3 "" H 1250 2300 50  0001 C CNN
+	1    1250 2300
+	1    0    0    -1
+$EndComp
+Wire Wire Line
+	2550 2100 2450 2100
+Wire Wire Line
+	2450 2100 2450 2350
+$Comp
+L power:GND #PWR02
+U 1 1 5D0819F7
+P 2450 2350
+F 0 "#PWR02" H 2450 2100 50  0001 C CNN
+F 1 "GND" H 2455 2177 50  0000 C CNN
+F 2 "" H 2450 2350 50  0001 C CNN
+F 3 "" H 2450 2350 50  0001 C CNN
+	1    2450 2350
+	1    0    0    -1
+$EndComp
+Wire Wire Line
+	5300 2200 5050 2200
+Wire Wire Line
+	5050 2200 5050 2400
+$Comp
+L power:GND #PWR04
+U 1 1 5D081A00
+P 5050 2400
+F 0 "#PWR04" H 5050 2150 50  0001 C CNN
+F 1 "GND" H 5055 2227 50  0000 C CNN
+F 2 "" H 5050 2400 50  0001 C CNN
+F 3 "" H 5050 2400 50  0001 C CNN
+	1    5050 2400
+	1    0    0    -1
+$EndComp
+Wire Wire Line
+	4150 2100 4400 2100
+Connection ~ 4400 2100
+Wire Wire Line
+	4400 2100 4750 2100
+Wire Wire Line
+	4400 2400 4600 2400
+Wire Wire Line
+	4600 2400 4600 2550
+Connection ~ 4600 2400
+Wire Wire Line
+	4600 2400 4750 2400
+$Comp
+L power:GND #PWR03
+U 1 1 5D081A0D
+P 4600 2550
+F 0 "#PWR03" H 4600 2300 50  0001 C CNN
+F 1 "GND" H 4605 2377 50  0000 C CNN
+F 2 "" H 4600 2550 50  0001 C CNN
+F 3 "" H 4600 2550 50  0001 C CNN
+	1    4600 2550
+	1    0    0    -1
+$EndComp
+Connection ~ 4750 2100
+Wire Wire Line
+	4750 2100 5300 2100
 $EndSCHEMATC
